File: PCB/right.kicad_sch (KiCad schematic)
At the start: 3 parts, among them J2 AudioJack4, U3 MCP23017_ML, U4 MOUDLE-SEEEDUINO-XIAO

Commit message: updated schematic
Parts:
- U3: symbol Interface_Expansion:MCP23017_ML -> Interface_Expansion:MCP23017_SP
Connections:
- net +3V3: now also U3.9 (VDD); no longer U3.5 (VDD)
- net GND: now also U3.10 (VSS); no longer U3.6 (VSS)
- net R_COL0: now also U3.21 (GPA0); no longer U3.17 (GPA0)
- net R_COL1: now also U3.22 (GPA1); no longer U3.18 (GPA1)
- net R_COL2: now also U3.23 (GPA2); no longer U3.19 (GPA2)
- net R_COL3: now also U3.24 (GPA3); no longer U3.20 (GPA3)
- net R_COL4: now also U3.25 (GPA4); no longer U3.21 (GPA4)
- net R_COL5: now also U3.26 (GPA5); no longer U3.22 (GPA5)
- net R_INT: now also U3.20 (INTA); no longer U3.16 (INTA)
- net R_ROW0: now also U3.1 (GPB0); no longer U3.25 (GPB0)
- net R_ROW1: now also U3.2 (GPB1); no longer U3.26 (GPB1)
- net R_ROW2: now also U3.3 (GPB2); no longer U3.27 (GPB2)
- net R_ROW3: now also U3.4 (GPB3); no longer U3.28 (GPB3)
- net R_ROW4: now also U3.5 (GPB4); no longer U3.1 (GPB4)
- net R_ROW5: now also U3.6 (GPB5); no longer U3.2 (GPB5)
- net R_ROW6: now also U3.7 (GPB6); no longer U3.3 (GPB6)
- net R_SCL_I2C1: now also U3.12 (SCK); no longer J2.S, U3.8 (SCK)
- net R_SDA_I2C1: now also U3.13 (SDA); no longer J2.R2, U3.9 (SDA)
- net R_SDA_I2C0: now reaches U4.7 (PB08_A6_D6_TX)
- net R_SDA_I2C0: now also J2.R2
- net R_SCL_I2C0: now reaches U4.8 (PB09_A7_D7_RX)
- net R_SCL_I2C0: now also J2.S
- new net R_COL6: U3.27 (GPA6)
- no-connect marks 0 -> 12
Other:
- note added: "IO Expander"
- note added: "MCU"
- note added: "TRRS Connector"
