File: PCB/split_keeb.kicad_pcb (KiCad board)
At the start: 2 copper layers, 3.6 x 3.3 mm, 248 parts, among them J1 AudioJack4, J2 AudioJack4, SW1 SW_Push, SW10 SW_Push, SW11 SW_Push, SW12 SW_Push, SW13 SW_Push, SW14 SW_Push, SW15 SW_Push, SW16 SW_Push, SW17 SW_Push, SW18 SW_Push, SW19 SW_Push, SW2 SW_Push, SW20 SW_Push, SW21 SW_Push, SW22 SW_Push, SW23 SW_Push, SW24 SW_Push, SW25 SW_Push, SW26 SW_Push, SW27 SW_Push, SW28 SW_Push, SW29 SW_Push, SW3 SW_Push, SW30 SW_Push, SW31 SW_Push, SW32 SW_Push, SW33 SW_Push, SW34 SW_Push, SW35 SW_Push, SW36 SW_Push, SW37 SW_Push, SW38 SW_Push, SW39 SW_Push, SW4 SW_Push, SW40 RotaryEncoder_Switch, SW41 SW_Push, SW42 SW_Push, SW43 SW_Push, SW44 SW_Push, SW45 SW_Push, SW46 SW_Push, SW47 SW_Push, SW48 SW_Push, SW49 SW_Push, SW5 SW_Push, SW50 SW_Push, SW51 SW_Push, SW52 SW_Push, SW53 SW_Push, SW54 SW_Push, SW55 SW_Push, SW56 SW_Push, SW57 SW_Push, SW58 SW_Push, SW59 SW_Push, SW6 SW_Push, SW60 SW_Push, SW61 SW_Push, SW62 SW_Push, SW63 SW_Push, SW64 SW_Push, SW65 SW_Push, SW66 SW_Push, SW67 SW_Push, SW68 SW_Push, SW69 SW_Push, SW7 SW_Push, SW70 SW_Push, SW71 SW_Push, SW72 SW_Push, SW73 SW_Push, SW74 SW_Push, SW75 SW_Push, SW76 SW_Push, SW77 SW_Push, SW78 SW_Push, SW79 SW_Push, SW8 SW_Push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

Commit message: updated schematic
Parts:
- moved D108 136.0 mm to (202.5, -4.30)
- moved D118 136.0 mm to (213.3, -4.30)
- moved D46 136.0 mm to (46.1, 6.24)
- moved D55 136.0 mm to (55.2, 6.24)
- moved D64 136.0 mm to (64.3, 6.24)
- moved D73 136.0 mm to (73.4, 6.24)
- moved D82 136.0 mm to (82.4, 6.24)
- moved D88 136.0 mm to (181.0, -4.30)
- moved D98 136.0 mm to (191.7, -4.30)
- moved D1 136.0 mm to (128.5, -113.9)
- moved D10 136.0 mm to (128.5, -81.9)
- moved D100 136.0 mm to (191.7, 2.80)
- moved D101 136.0 mm to (191.7, 6.35)
- moved D102 136.0 mm to (191.7, 9.90)
- moved D103 136.0 mm to (202.5, -22.1)
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
Commit message: routed the switches and diodes
Parts:
- removed D122, D123, D124, D125, D126, D127, D128, D129, D130, D131, D132, D133, D134, D135, D136, D137, D138, D139, D140, D141, D142, D143, D144, D145, D146, D147, D148, D149, D150, D151, D152, D153, D154, D155, D156, D157, D158, D159, D160, D161, D162, D163, D41, D42, D43, D44, D45, D46, D47, D48, D49, D50, D51, D52, D53, D54, D55, D56, D57, D58, D59, D60, D61, D62, D63, D64, D65, D66, D67, D68, D69, D70, D71, D72, D73, D74, D75, D76, D77, D78, D79, D80, D81, D82: SK6812MINI-E, footprints:SK6812MINI-E_fixed
- SW15, SW21, SW27, SW33, SW66, SW72: footprint Gateron_KS33_Hotswap:Gateron-KS33-Hotswap-1U -> Gateron_KS33_Hotswap:Gateron-KS33-Hotswap-1.25U
- SW23, SW24, SW35, SW76, SW79: footprint Gateron_KS33_Hotswap:Gateron-KS33-Hotswap-1.25U -> Gateron_KS33_Hotswap:Gateron-KS33-Hotswap-1U
- SW30, SW39, SW61: footprint Gateron_KS33_Hotswap:Gateron-KS33-Hotswap-2U -> Gateron_KS33_Hotswap:Gateron-KS33-Hotswap-1U
- SW36, SW78: footprint Gateron_KS33_Hotswap:Gateron-KS33-Hotswap-1.25U -> Gateron_KS33_Hotswap:Gateron-KS33-Hotswap-2U
- SW38, SW73: footprint Gateron_KS33_Hotswap:Gateron-KS33-Hotswap-1U -> Gateron_KS33_Hotswap:Gateron-KS33-Hotswap-2U
- SW60: footprint Gateron_KS33_Hotswap:Gateron-KS33-Hotswap-2U -> Gateron_KS33_Hotswap:Gateron-KS33-Hotswap-1.25U
- moved SW73 271.1 mm to (192.5, 151.0), turned to 120 degrees
- moved SW74 267.1 mm to (171.2, 152.3), turned to 30 degrees
- moved SW78 242.5 mm to (198.5, 180.5), turned to 30 degrees
- moved SW75 231.7 mm to (269.5, 141.5)
- moved SW79 225.2 mm to (180.7, 168.8), turned to 30 degrees
- moved SW76 222.3 mm to (288.5, 141.5)
- moved SW65 222.1 mm to (288.5, 103.5)
- moved SW66 217.0 mm to (310.0, 103.5)
- moved SW77 215.4 mm to (310.0, 141.5)
- moved SW67 213.8 mm to (212.5, 122.5)
- moved U3 213.8 mm to (371.9, 120.6)
- moved J2 210.3 mm to (389.2, 144.2), turned to -90 degrees
- moved U4 208.1 mm to (355.8, 141.2)
- moved SW68 200.9 mm to (231.5, 122.5)
- moved SW57 199.3 mm to (250.5, 84.5)
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Connections:
- D100 pad 1: R_ROW3 -> R_ROW2
- D101 pad 1: R_ROW4 -> R_ROW2
- D102 pad 1: R_ROW5 -> R_ROW2
- D103 pad 1: R_ROW6 -> R_ROW3
- D104 pad 1: R_ROW0 -> R_ROW3
- D105 pad 1: R_ROW1 -> R_ROW3
- D106 pad 1: R_ROW2 -> R_ROW3
- D108 pad 1: R_ROW4 -> R_ROW3
- D109 pad 1: R_ROW5 -> R_ROW4
- D110 pad 1: R_ROW0 -> R_ROW4
- D111 pad 1: R_ROW1 -> R_ROW4
- D112 pad 1: R_ROW2 -> R_ROW4
- D113 pad 1: R_ROW3 -> R_ROW4
- D116 pad 1: R_ROW0 -> R_ROW5
- D117 pad 1: R_ROW1 -> R_ROW5
- D118 pad 1: R_ROW2 -> R_ROW5
- D119 pad 1: R_ROW3 -> R_ROW5
- D120 pad 1: R_ROW4 -> R_ROW6
- D121 pad 1: R_ROW5 -> R_ROW6
- D13 pad 1: L_ROW2 -> L_ROW1
- D14 pad 1: L_ROW3 -> L_ROW1
- D16 pad 1: L_ROW3 -> L_ROW2
- D18 pad 1: L_ROW3 -> L_ROW2
- D20 pad 1: L_ROW3 -> L_ROW2
- D21 pad 1: L_ROW2 -> L_ROW3
- D23 pad 1: L_ROW2 -> L_ROW3
- D25 pad 1: L_ROW4 -> L_ROW3
- D26 pad 1: L_ROW5 -> L_ROW3
- D28 pad 1: L_ROW5 -> L_ROW4
- D30 pad 1: L_ROW5 -> L_ROW4
- D32 pad 1: L_ROW5 -> L_ROW4
- D33 pad 1: L_ROW4 -> L_ROW5
- D35 pad 1: L_ROW4 -> L_ROW5
- D37 pad 1: L_ROW6 -> L_ROW5
- D7 pad 1: L_ROW1 -> L_ROW0
- D84 pad 1: R_ROW1 -> R_ROW0
- D85 pad 1: R_ROW2 -> R_ROW0
- D86 pad 1: R_ROW3 -> R_ROW0
- D87 pad 1: R_ROW4 -> R_ROW0
- D88 pad 1: R_ROW5 -> R_ROW0
- D89 pad 1: R_ROW6 -> R_ROW0
- D90 pad 1: R_ROW0 -> R_ROW1
- D92 pad 1: R_ROW2 -> R_ROW1
- D93 pad 1: R_ROW3 -> R_ROW1
- D94 pad 1: R_ROW4 -> R_ROW1
- D95 pad 1: R_ROW5 -> R_ROW1
- D96 pad 1: R_ROW6 -> R_ROW1
- D97 pad 1: R_ROW0 -> R_ROW2
- D98 pad 1: R_ROW1 -> R_ROW2
- J1 pad R2: L_SDA_I2C0 -> L_SDA_I2C1
- J1 pad S: L_SCL_I2C0 -> L_SCL_I2C1
- J2 pad R2: R_SDA_I2C1 -> R_SDA_I2C0
- J2 pad S: R_SCL_I2C1 -> R_SCL_I2C0
- SW10 pad 1: L_COL3 -> L_COL2
- SW11 pad 1: L_COL4 -> L_COL3
- SW12 pad 1: L_COL5 -> L_COL4
- SW13 pad 1: L_COL0 -> L_COL5
- SW14 pad 1: L_COL0 -> L_COL6
- SW15 pad 1: L_COL1 -> L_COL0
- SW18 pad 1: L_COL2 -> L_COL3
- SW19 pad 1: L_COL3 -> L_COL4
- SW20 pad 1: L_COL3 -> L_COL5
- SW21 pad 1: L_COL4 -> L_COL0
- SW22 pad 1: L_COL4 -> L_COL1
- SW23 pad 1: L_COL5 -> L_COL2
- SW24 pad 1: L_COL5 -> L_COL3
- SW25 pad 1: L_COL0 -> L_COL4
- SW26 pad 1: L_COL0 -> L_COL5
- SW27 pad 1: L_COL1 -> L_COL0
- SW30 pad 1: L_COL2 -> L_COL3
- SW31 pad 1: L_COL3 -> L_COL4
- SW32 pad 1: L_COL3 -> L_COL5
- SW33 pad 1: L_COL4 -> L_COL0
- SW34 pad 1: L_COL4 -> L_COL1
- SW35 pad 1: L_COL5 -> L_COL2
- SW37 pad 1: L_COL0 -> L_COL6
- SW38 pad 1: L_COL1 -> L_COL5
- SW39 pad 1: L_COL2 -> L_COL6
- SW40 pad A: Net-(D40-A) -> L_COL0
- SW40 pad B: L_COL3 -> Net-(D40-A)
- SW40 pad S1: L_ENCA -> L_ENCB
- SW40 pad S2: L_ENCB -> L_ENCA
- SW42 pad 1: R_COL0 -> R_COL1
- SW43 pad 1: R_COL0 -> R_COL2
- SW44 pad 1: R_COL0 -> R_COL3
- SW45 pad 1: R_COL0 -> R_COL4
- SW46 pad 1: R_COL0 -> R_COL5
- SW47 pad 1: R_COL0 -> R_COL6
- SW48 pad 1: R_COL1 -> R_COL0
- SW50 pad 1: R_COL1 -> R_COL2
- SW51 pad 1: R_COL1 -> R_COL3
- SW52 pad 1: R_COL1 -> R_COL4
- SW53 pad 1: R_COL1 -> R_COL5
- SW54 pad 1: R_COL1 -> R_COL6
- SW55 pad 1: R_COL2 -> R_COL1
- SW57 pad 1: R_COL2 -> R_COL3
- SW58 pad 1: R_COL2 -> R_COL4
- SW59 pad 1: R_COL2 -> R_COL5
- SW60 pad 1: R_COL2 -> R_COL6
- SW61 pad 1: R_COL2 -> R_COL1
- SW62 pad 1: R_COL3 -> R_COL2
- SW64 pad 1: R_COL3 -> R_COL4
- SW65 pad 1: R_COL3 -> R_COL5
- SW66 pad 1: R_COL3 -> R_COL6
- SW67 pad 1: R_COL3 -> R_COL1
- SW68 pad 1: R_COL4 -> R_COL2
- SW69 pad 1: R_COL4 -> R_COL3
- SW7 pad 1: L_COL0 -> L_COL6
- SW71 pad 1: R_COL4 -> R_COL5
- SW72 pad 1: R_COL4 -> R_COL6
- SW73 pad 1: R_COL4 -> R_COL0
- SW74 pad 1: R_COL5 -> R_COL1
- SW75 pad 1: R_COL5 -> R_COL4
- SW77 pad 1: R_COL5 -> R_COL6
- SW78 pad 1: R_COL5 -> R_COL0
- SW79 pad 1: R_COL5 -> R_COL1
- SW8 pad 1: L_COL1 -> L_COL0
- SW9 pad 1: L_COL2 -> L_COL1
- U1 pad 7: L_SDA_I2C0 -> unconnected-(U1-PB08_A6_D6_TX-Pad7)
- U1 pad 8: L_SCL_I2C0 -> unconnected-(U1-PB09_A7_D7_RX-Pad8)
- U2 pad 1: L_ROW4 -> L_ROW0
- U2 pad 10: unconnected-(U2-NC-Pad10) -> GND
- U2 pad 12: unconnected-(U2-A1-Pad12) -> L_SCL_I2C1
- U2 pad 13: unconnected-(U2-A2-Pad13) -> L_SDA_I2C1
- U2 pad 16: L_INT -> unconnected-(U2-A1-Pad16)
- U2 pad 17: L_COL0 -> unconnected-(U2-A2-Pad17)
- U2 pad 18: L_COL1 -> unconnected-(U2-~{RESET}-Pad18)
- U2 pad 19: L_COL2 -> unconnected-(U2-INTB-Pad19)
- U2 pad 2: L_ROW5 -> L_ROW1
- U2 pad 20: L_COL3 -> L_INT
- U2 pad 21: L_COL4 -> L_COL0
- U2 pad 22: L_COL5 -> L_COL1
- U2 pad 23: unconnected-(U2-GPA6-Pad23) -> L_COL2
- U2 pad 24: unconnected-(U2-GPA7-Pad24) -> L_COL3
- U2 pad 25: L_ROW0 -> L_COL4
- U2 pad 26: L_ROW1 -> L_COL5
- U2 pad 27: L_ROW2 -> L_COL6
- U2 pad 28: L_ROW3 -> unconnected-(U2-GPA7-Pad28)
- U2 pad 3: L_ROW6 -> L_ROW2
- U2 pad 4: unconnected-(U2-GPB7-Pad4) -> L_ROW3
- U2 pad 5: +3V3 -> L_ROW4
- U2 pad 6: GND -> L_ROW5
- U2 pad 7: unconnected-(U2-NC-Pad7) -> L_ROW6
- U2 pad 8: L_SCL_I2C1 -> unconnected-(U2-GPB7-Pad8)
- U2 pad 9: L_SDA_I2C1 -> +3V3
- U3 pad 1: R_ROW4 -> R_ROW0
- U3 pad 10: unconnected-(U3-NC-Pad10) -> GND
- U3 pad 12: unconnected-(U3-A1-Pad12) -> R_SCL_I2C1
- U3 pad 13: unconnected-(U3-A2-Pad13) -> R_SDA_I2C1
- U3 pad 16: R_INT -> unconnected-(U3-A1-Pad16)
- U3 pad 17: R_COL0 -> unconnected-(U3-A2-Pad17)
- U3 pad 18: R_COL1 -> unconnected-(U3-~{RESET}-Pad18)
- U3 pad 19: R_COL2 -> unconnected-(U3-INTB-Pad19)
- U3 pad 2: R_ROW5 -> R_ROW1
- U3 pad 20: R_COL3 -> R_INT
- U3 pad 21: R_COL4 -> R_COL0
- U3 pad 22: R_COL5 -> R_COL1
- U3 pad 23: unconnected-(U3-GPA6-Pad23) -> R_COL2
- U3 pad 24: unconnected-(U3-GPA7-Pad24) -> R_COL3
- U3 pad 25: R_ROW0 -> R_COL4
- U3 pad 26: R_ROW1 -> R_COL5
- U3 pad 27: R_ROW2 -> R_COL6
- U3 pad 28: R_ROW3 -> unconnected-(U3-GPA7-Pad28)
- U3 pad 3: R_ROW6 -> R_ROW2
- U3 pad 4: unconnected-(U3-GPB7-Pad4) -> R_ROW3
- U3 pad 5: +3V3 -> R_ROW4
- U3 pad 6: GND -> R_ROW5
- U3 pad 7: unconnected-(U3-NC-Pad7) -> R_ROW6
- U3 pad 8: R_SCL_I2C1 -> unconnected-(U3-GPB7-Pad8)
- U3 pad 9: R_SDA_I2C1 -> +3V3
- U4 pad 7: unconnected-(U4-PB08_A6_D6_TX-Pad7) -> R_SDA_I2C0
- U4 pad 8: unconnected-(U4-PB09_A7_D7_RX-Pad8) -> R_SCL_I2C0
Routing:
- net R_COL1: track 0.00 -> 158.4 mm, vias 0 -> 12
- net R_COL0: track 0.00 -> 145.7 mm, vias 0 -> 6
- net R_ROW5: track 0.00 -> 144.7 mm, vias 0 -> 1
- net R_ROW1: track 0.00 -> 119.5 mm
- net R_ROW0: track 0.00 -> 119.4 mm
- net R_COL4: track 0.00 -> 102.9 mm, vias 0 -> 10
- net R_COL5: track 0.00 -> 102.7 mm, vias 0 -> 10
- net R_ROW4: track 0.00 -> 102.4 mm
- net R_ROW3: track 0.00 -> 102.1 mm
- net R_ROW2: track 0.00 -> 101.9 mm
- net R_COL6: track 0.00 -> 99.8 mm
- net R_COL3: track 0.00 -> 83.7 mm, vias 0 -> 8
- net R_COL2: track 0.00 -> 83.7 mm, vias 0 -> 8
- net R_ROW6: track 0.00 -> 22.4 mm
- net Net-(D120-A): track 0.00 -> 12.8 mm
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Other:
- board outline removed

Commit message: "finished" right side
Parts:
- added D122: SK6812MINI-E, footprints:SK6812MINI-E_fixed, F.Cu at (136.4, -10.4)
- added D123: SK6812MINI-E, footprints:SK6812MINI-E_fixed, F.Cu at (136.4, -5.35)
- added D124: SK6812MINI-E, footprints:SK6812MINI-E_fixed, F.Cu at (136.4, -0.30)
- added D125: SK6812MINI-E, footprints:SK6812MINI-E_fixed, F.Cu at (136.4, 4.75)
- added D126: SK6812MINI-E, footprints:SK6812MINI-E_fixed, F.Cu at (136.4, 9.80)
- added D127: SK6812MINI-E, footprints:SK6812MINI-E_fixed, F.Cu at (136.4, 14.9)
- added D128: SK6812MINI-E, footprints:SK6812MINI-E_fixed, F.Cu at (145.5, -30.6)
- added D129: SK6812MINI-E, footprints:SK6812MINI-E_fixed, F.Cu at (145.5, -25.5)
- added D130: SK6812MINI-E, footprints:SK6812MINI-E_fixed, F.Cu at (145.5, -20.5)
- added D131: SK6812MINI-E, footprints:SK6812MINI-E_fixed, F.Cu at (145.5, -15.4)
- added D132: SK6812MINI-E, footprints:SK6812MINI-E_fixed, F.Cu at (145.5, -10.4)
- added D133: SK6812MINI-E, footprints:SK6812MINI-E_fixed, F.Cu at (145.5, -5.35)
- added D134: SK6812MINI-E, footprints:SK6812MINI-E_fixed, F.Cu at (145.5, -0.30)
- added D135: SK6812MINI-E, footprints:SK6812MINI-E_fixed, F.Cu at (145.5, 4.75)
- added D136: SK6812MINI-E, footprints:SK6812MINI-E_fixed, F.Cu at (145.5, 9.80)
- added D137: SK6812MINI-E, footprints:SK6812MINI-E_fixed, F.Cu at (145.5, 14.9)
- added D138: SK6812MINI-E, footprints:SK6812MINI-E_fixed, F.Cu at (154.6, -30.6)
- added D139: SK6812MINI-E, footprints:SK6812MINI-E_fixed, F.Cu at (154.6, -25.5)
- added D140: SK6812MINI-E, footprints:SK6812MINI-E_fixed, F.Cu at (154.6, -20.5)
- added D141: SK6812MINI-E, footprints:SK6812MINI-E_fixed, F.Cu at (154.6, -15.4)
- added D142: SK6812MINI-E, footprints:SK6812MINI-E_fixed, F.Cu at (154.6, -10.4)
- added D143: SK6812MINI-E, footprints:SK6812MINI-E_fixed, F.Cu at (154.6, -5.35)
- added D144: SK6812MINI-E, footprints:SK6812MINI-E_fixed, F.Cu at (154.6, -0.30)
- added D145: SK6812MINI-E, footprints:SK6812MINI-E_fixed, F.Cu at (154.6, 4.75)
- added D146: SK6812MINI-E, footprints:SK6812MINI-E_fixed, F.Cu at (154.6, 9.80)
- added D147: SK6812MINI-E, footprints:SK6812MINI-E_fixed, F.Cu at (154.6, 14.9)
- added D148: SK6812MINI-E, footprints:SK6812MINI-E_fixed, F.Cu at (163.7, -30.6)
- added D149: SK6812MINI-E, footprints:SK6812MINI-E_fixed, F.Cu at (163.7, -25.5)
- added D150: SK6812MINI-E, footprints:SK6812MINI-E_fixed, F.Cu at (163.7, -20.5)
- added D151: SK6812MINI-E, footprints:SK6812MINI-E_fixed, F.Cu at (163.7, -15.4)
- added D152: SK6812MINI-E, footprints:SK6812MINI-E_fixed, F.Cu at (163.7, -10.4)
- added D153: SK6812MINI-E, footprints:SK6812MINI-E_fixed, F.Cu at (163.7, -5.35)
- added D154: SK6812MINI-E, footprints:SK6812MINI-E_fixed, F.Cu at (163.7, -0.30)
- added D155: SK6812MINI-E, footprints:SK6812MINI-E_fixed, F.Cu at (163.7, 4.75)
- added D156: SK6812MINI-E, footprints:SK6812MINI-E_fixed, B.Cu at (178.7, 164.3)
- added D157: SK6812MINI-E, footprints:SK6812MINI-E_fixed, F.Cu at (163.4, 16.9)
- added D41: SK6812MINI-E, footprints:SK6812MINI-E_fixed, B.Cu at (190.0, 41.5)
- added D42: SK6812MINI-E, footprints:SK6812MINI-E_fixed, B.Cu at (209.0, 41.5)
- added D43: SK6812MINI-E, footprints:SK6812MINI-E_fixed, B.Cu at (228.0, 41.5)
- added D44: SK6812MINI-E, footprints:SK6812MINI-E_fixed, B.Cu at (246.5, 41.5)
- added D45: SK6812MINI-E, footprints:SK6812MINI-E_fixed, B.Cu at (266.0, 41.5)
- added D46: SK6812MINI-E, footprints:SK6812MINI-E_fixed, B.Cu at (285.0, 41.5)
- added D47: SK6812MINI-E, footprints:SK6812MINI-E_fixed, B.Cu at (304.0, 41.5)
- added D48: SK6812MINI-E, footprints:SK6812MINI-E_fixed, B.Cu at (199.0, 60.5)
- added D49: SK6812MINI-E, footprints:SK6812MINI-E_fixed, B.Cu at (218.0, 60.5)
- added D50: SK6812MINI-E, footprints:SK6812MINI-E_fixed, B.Cu at (237.0, 60.5)
- added D51: SK6812MINI-E, footprints:SK6812MINI-E_fixed, B.Cu at (255.9, 60.5)
- added D52: SK6812MINI-E, footprints:SK6812MINI-E_fixed, B.Cu at (275.0, 60.5)
- added D53: SK6812MINI-E, footprints:SK6812MINI-E_fixed, B.Cu at (294.0, 60.5)
- added D54: SK6812MINI-E, footprints:SK6812MINI-E_fixed, B.Cu at (313.0, 60.5)
- added D55: SK6812MINI-E, footprints:SK6812MINI-E_fixed, B.Cu at (213.0, 79.5)
- added D56: SK6812MINI-E, footprints:SK6812MINI-E_fixed, B.Cu at (232.0, 79.5)
- added D57: SK6812MINI-E, footprints:SK6812MINI-E_fixed, B.Cu at (251.0, 79.5)
- added D58: SK6812MINI-E, footprints:SK6812MINI-E_fixed, B.Cu at (270.0, 79.5)
- added D59: SK6812MINI-E, footprints:SK6812MINI-E_fixed, B.Cu at (289.0, 79.5)
- added D60: SK6812MINI-E, footprints:SK6812MINI-E_fixed, B.Cu at (310.5, 79.5)
- added D61: SK6812MINI-E, footprints:SK6812MINI-E_fixed, B.Cu at (213.0, 98.5)
- added D62: SK6812MINI-E, footprints:SK6812MINI-E_fixed, B.Cu at (232.0, 98.5)
- added D63: SK6812MINI-E, footprints:SK6812MINI-E_fixed, B.Cu at (251.0, 98.5)
- added D64: SK6812MINI-E, footprints:SK6812MINI-E_fixed, B.Cu at (270.0, 98.5)
- added D65: SK6812MINI-E, footprints:SK6812MINI-E_fixed, B.Cu at (289.0, 98.5)
- added D66: SK6812MINI-E, footprints:SK6812MINI-E_fixed, B.Cu at (310.5, 98.5)
- added D67: SK6812MINI-E, footprints:SK6812MINI-E_fixed, B.Cu at (213.0, 117.5)
- added D68: SK6812MINI-E, footprints:SK6812MINI-E_fixed, B.Cu at (232.0, 117.5)
- added D69: SK6812MINI-E, footprints:SK6812MINI-E_fixed, B.Cu at (251.0, 117.5)
- added D70: SK6812MINI-E, footprints:SK6812MINI-E_fixed, B.Cu at (270.0, 117.5)
- added D71: SK6812MINI-E, footprints:SK6812MINI-E_fixed, B.Cu at (288.9, 117.5)
- added D72: SK6812MINI-E, footprints:SK6812MINI-E_fixed, B.Cu at (310.5, 117.5)
- added D73: SK6812MINI-E, footprints:SK6812MINI-E_fixed, B.Cu at (188.0, 153.0)
- added D74: SK6812MINI-E, footprints:SK6812MINI-E_fixed, B.Cu at (169.2, 147.7)
- added D75: SK6812MINI-E, footprints:SK6812MINI-E_fixed, B.Cu at (270.0, 136.5)
- added D76: SK6812MINI-E, footprints:SK6812MINI-E_fixed, B.Cu at (289.0, 136.5)
- added D77: SK6812MINI-E, footprints:SK6812MINI-E_fixed, B.Cu at (310.5, 136.5)
- added D78: SK6812MINI-E, footprints:SK6812MINI-E_fixed, B.Cu at (196.5, 176.0)
- added D79: SK6812MINI-E, footprints:SK6812MINI-E_fixed, F.Cu at (136.5, -30.5)
- added D80: SK6812MINI-E, footprints:SK6812MINI-E_fixed, F.Cu at (136.4, -25.5)
- added D81: SK6812MINI-E, footprints:SK6812MINI-E_fixed, F.Cu at (136.4, -20.5)
- added D82: SK6812MINI-E, footprints:SK6812MINI-E_fixed, F.Cu at (136.4, -15.4)
- J2: moved to B.Cu
- moved J2 262.4 mm to (149.5, 37.5)
- moved U4 215.2 mm to (165.4, 40.9)
- moved U3 203.4 mm to (171.2, 87.5)
Routing:
- net GND: track 0.00 -> 1312.7 mm, vias 0 -> 82
- net VCC: track 0.00 -> 1063.1 mm, vias 0 -> 50
- net R_COL6: track 99.8 -> 296.7 mm, vias 0 -> 4
- net R_COL5: track 102.7 -> 283.8 mm, vias 10 -> 16
- net R_COL4: track 102.9 -> 269.0 mm, vias 10 -> 15
- net Net-(D72-DOUT): track 0.00 -> 165.6 mm, vias 0 -> 2
- net R_COL3: track 83.7 -> 232.9 mm, vias 8 -> 12
- net Net-(D77-DOUT): track 0.00 -> 146.0 mm, vias 0 -> 4
- net R_INT: track 0.00 -> 142.7 mm, vias 0 -> 4
- net R_COL2: track 83.7 -> 220.5 mm, vias 8 -> 13
- net R_ROW5: track 144.7 -> 279.0 mm, vias 1 -> 3
- net R_SCL_I2C1: track 0.00 -> 131.1 mm, vias 0 -> 2
- net +3V3: track 0.00 -> 128.8 mm, vias 0 -> 4
- net Net-(D47-DOUT): track 0.00 -> 127.2 mm, vias 0 -> 2
- net R_SDA_I2C1: track 0.00 -> 124.2 mm, vias 0 -> 2
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Other:
- board outline added: 181.5 x 171.7 mm

Commit message: wired up leds and matrix for left
Parts:
- D156, D41, D42, D43, D44, D45, D46, D47, D48, D49, D50, D51, D52, D53, D54, D55, D56, D57, D58, D59, D60, D61, D62, D63, D64, D65, D66, D67, D68, D69, D70, D71, D72, D73, D74, D75, D76, D77, D78, J2: moved to F.Cu
- SW1, SW10, SW11, SW12, SW13, SW14, SW16, SW17, SW18, SW19, SW2, SW20, SW22, SW23, SW24, SW25, SW26, SW28, SW29, SW3, SW30, SW31, SW32, SW34, SW35, SW37, SW39, SW4, SW41, SW42, SW43, SW44, SW45, SW46, SW47, SW48, SW49, SW5, SW50, SW51, SW52, SW53, SW54, SW55, SW56, SW57, SW58, SW59, SW6, SW61, SW62, SW63, SW64, SW65, SW67, SW68, SW69, SW7, SW70, SW71, SW74, SW75, SW76, SW79, SW8, SW9: footprint Gateron_KS33_Hotswap:Gateron-KS33-Hotswap-1U -> PCM_marbastlib-xp-gateron_lp:SW_KS33_HS_KS-2P02B01-02_HS_1u; moved to B.Cu
- SW15, SW21, SW27, SW33, SW60, SW66, SW72, SW77: footprint Gateron_KS33_Hotswap:Gateron-KS33-Hotswap-1.25U -> PCM_marbastlib-xp-gateron_lp:SW_KS33_HS_KS-2P02B01-02_1.25u; moved to B.Cu
- SW36, SW38, SW73, SW78: footprint Gateron_KS33_Hotswap:Gateron-KS33-Hotswap-2U -> PCM_marbastlib-xp-gateron_lp:SW_KS33_HS_KS-2P02B01-02_1.75u; moved to B.Cu
- moved SW73 427.2 mm to (48.1, -251.0), turned to 180 degrees
- moved D120 425.0 mm to (170.6, -233.2), turned to 0 degrees
- moved SW75 422.9 mm to (48.1, -218.8), turned to 180 degrees
- moved SW76 419.9 mm to (48.1, -202.7), turned to 180 degrees
- moved SW77 419.8 mm to (48.1, -186.6), turned to 180 degrees
- moved SW65 418.9 mm to (65.4, -251.0), turned to 180 degrees
- moved SW66 417.5 mm to (65.4, -234.9), turned to 180 degrees
- moved D119 410.7 mm to (170.6, -236.8)
- moved D116 409.8 mm to (170.6, -247.4), turned to 0 degrees
- moved D114 409.5 mm to (170.6, -254.6)
- moved D121 408.7 mm to (170.6, -229.7), turned to 0 degrees
- moved D118 407.5 mm to (170.6, -240.3)
- moved D113 406.4 mm to (170.6, -258.1)
- moved SW74 406.3 mm to (48.1, -234.9), turned to 180 degrees
- moved D117 406.1 mm to (170.6, -243.9)
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Routing:
- net R_COL6: track 296.7 -> 0.00 mm, vias 4 -> 0
- net R_COL5: track 283.8 -> 0.00 mm, vias 16 -> 0
- net R_ROW5: track 279.0 -> 0.00 mm, vias 3 -> 0
- net R_COL4: track 269.0 -> 0.00 mm, vias 15 -> 0
- net R_COL1: track 251.7 -> 0.00 mm, vias 16 -> 0
- net R_COL3: track 232.9 -> 0.00 mm, vias 12 -> 0
- net R_COL2: track 220.5 -> 0.00 mm, vias 13 -> 0
- net R_COL0: track 220.1 -> 0.00 mm, vias 11 -> 0
- net R_ROW4: track 173.8 -> 0.00 mm, vias 2 -> 0
- net Net-(D72-DOUT): track 165.6 -> 0.00 mm, vias 2 -> 0
- net L_COL5: track 0.00 -> 162.0 mm
- net R_ROW0: track 156.8 -> 0.00 mm
- net L_ROW5: track 0.00 -> 153.6 mm, vias 0 -> 1
- net R_ROW3: track 151.7 -> 0.00 mm, vias 1 -> 0
- net R_ROW1: track 148.9 -> 0.00 mm
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Other:
- board size 181.5 x 171.7 mm -> 187 x 175 mm
